Commit message: Hook and drop process added

File: src/arm_only/config/gazebo_feetech.urdf (robot description, URDF)
Before this commit: robot feetech, 9 links, 8 joints
Links:
- added link realsense_link, mass 0.072; collision box size=0.09 0.025 0.025; visual mesh filename=package://realsense2_description/meshes/d435.dae
- added link realsense_optical_frame
Joints:
- added joint realsense_joint: type fixed, parent base_link, child realsense_link, origin xyz=0.04 0 0 rpy=0 0 0
- added joint realsense_optical_joint: type fixed, parent realsense_link, child realsense_optical_frame, origin xyz=0 0 0 rpy=-1.5708 0 -1.5708
- joint world_joint: origin xyz=0 0 1 rpy=0 0 0 -> xyz=0 0 0.5 rpy=0 0 0
